Commit message: fix: URDF joint axis Z→Y and add pto_joint to JointState for RViz
Agent-Logs-Url: https://github.com/salhus/hil_odrive_chrono_ros2_control/sessions/ea860146-0cf8-4842-8b01-d829fbd25be2

Co-authored-by: salhus <84348506+salhus@users.noreply.github.com>

File: src/hil_odrive_ros2_control/description/urdf/motor.urdf.xacro (robot description, xacro)
@@ -38,5 +38,5 @@
     <child link="motor_link"/>
     <origin xyz="0 0 0" rpy="0 0 0"/>
-    <axis xyz="0 0 1"/>
+    <axis xyz="0 1 0"/>
   </joint>
   <!-- PTO motor (axis1) — same shaft as motor_joint, passive linear damper -->
@@ -55,5 +55,5 @@
     <child link="pto_link"/>
     <origin xyz="0 0 0" rpy="0 0 0"/>
-    <axis xyz="0 0 1"/>
+    <axis xyz="0 1 0"/>
   </joint>
   <!-- ros2_control hardware — both axes on the same ODrive board / CAN bus -->

Commit message: fix: swap flap visual box X/Y dimensions for correct Y-axis rotation orientation
Agent-Logs-Url: https://github.com/salhus/hil_odrive_chrono_ros2_control/sessions/d25ac848-210b-41d0-aa8b-482f791bd769

Co-authored-by: salhus <84348506+salhus@users.noreply.github.com>

File: src/hil_odrive_ros2_control/description/urdf/motor.urdf.xacro (robot description, xacro)
@@ -12,5 +12,5 @@
     </visual>
   </link>
-  <!-- 30cm wide x 0.25cm thick x 30cm tall acrylic flap (width x thickness x height) -->
+  <!-- 0.25cm thick x 30cm wide x 30cm tall acrylic flap (thickness x width x height) -->
   <!-- CoM is at z=0.15 (half of 0.30m height) above the joint origin -->
   <link name="motor_link">
@@ -18,6 +18,6 @@
       <origin xyz="0 0 0.15" rpy="0 0 0"/>
       <geometry>
-        <!-- size: x=0.30m (width), y=0.0025m (thickness), z=0.30m (height) -->
-        <box size="0.30 0.0025 0.30"/>
+        <!-- size: x=0.0025m (thickness), y=0.30m (width along rotation axis), z=0.30m (height) -->
+        <box size="0.0025 0.30 0.30"/>
       </geometry>
       <material name="acrylic_blue">
